File: tally_lanc.kicad_pcb (KiCad board)
At the start: 2 copper layers, 50.8 x 25.4 mm, 16 parts, among them J1 Conn_01x05, J2 Conn_01x03, J3 Conn_01x12, J4 LANC Out, J5 LANC In, Q1 BC547

Commit message: V2.0
Parts:
- J4, J5: footprint GJK Footprints:jack_2.5mm_trs -> GJK Footprints 1:jack_2.5mm_trs_smd
- REF** (x2): moved to B.Cu
- moved REF** 37.9 mm to (74.0, 85.0), turned to 180 degrees
- moved REF** 35.2 mm to (76.0, 96.0), turned to 180 degrees
- moved R1 4.04 mm to (81.5, 81.5)
- moved D1 3.79 mm to (84.5, 89.3)
- moved J5 1.52 mm to (74.0, 95.0)
- moved J4 1.18 mm to (74.0, 85.0)
Routing:
- net GND: track 0.00 -> 22.7 mm
- net Net-(D1-K): track 37.6 -> 22.1 mm
- net Net-(R1-+): track 16.0 -> 21.8 mm
Other:
- board size 50.8 x 25.4 mm -> 40.4 x 25.4 mm
- board text added: "Tally Arbiter TTGO_T LANC interface V2 Designed by Peter de Jonge & Gert Jan Kruizinga"
- board text removed: "Tally Arbiter TTGO_T LANC interface Designed by Peter de Jonge & Gert Jan Kruizinga"
