File: tally_lanc.kicad_sch (KiCad schematic)
At the start: 14 parts, among them J1 Conn_01x05, J2 Conn_01x03, J3 Conn_01x12, J4 LANC Out, J5 LANC In, Q1 BC547

Commit message: V2.0
Parts:
- J4, J5: footprint GJK Footprints:jack_2.5mm_trs -> GJK Footprints 1:jack_2.5mm_trs_smd
Changed lines of the file:
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@@
 (kicad_sch
-	(version 20231120)
+	(version 20250114)
 	(generator "eeschema")
-	(generator_version "8.0")
+	(generator_version "9.0")
 	(paper "A4")
 	(title_block
@@
 	(label "Red"
 		(at 55.88 91.44 0)
-		(fields_autoplaced yes)
 		(effects
 			(font
@@
 	(label "Green"
 		(at 55.88 93.98 0)
-		(fields_autoplaced yes)
 		(effects
 			(font
@@
 	(label "Green"
 		(at 106.68 96.52 180)
-		(fields_autoplaced yes)
 		(effects
 			(font
@@
 	(label "lanc_rx"
 		(at 55.88 99.06 0)
-		(fields_autoplaced yes)
 		(effects
 			(font
@@
 	(label "lanc_rx"
 		(at 111.76 50.8 180)
-		(fields_autoplaced yes)
 		(effects
 			(font
@@
 	(label "Blue"
 		(at 106.68 101.6 180)
-		(fields_autoplaced yes)
 		(effects
 			(font
@@
 	(label "lanc_tx"
 		(at 111.76 60.96 180)
-		(fields_autoplaced yes)
 		(effects
 			(font
@@
 	(label "Red"
 		(at 106.68 91.44 180)
-		(fields_autoplaced yes)
 		(effects
 			(font
@@
 	(label "lanc_tx"
 		(at 55.88 101.6 0)
-		(fields_autoplaced yes)
 		(effects
 			(font
@@
 	(label "Blue"
 		(at 55.88 96.52 0)
-		(fields_autoplaced yes)
 		(effects
 			(font
@@
 			)
 		)
-		(property "Footprint" "GJK Footprints:jack_2.5mm_trs"
+		(property "Footprint" "GJK Footprints 1:jack_2.5mm_trs_smd"
 			(at 160.02 78.74 0)
 			(effects
@@
 			)
 		)
-		(property "Footprint" "GJK Footprints:jack_2.5mm_trs"
+		(property "Footprint" "GJK Footprints 1:jack_2.5mm_trs_smd"
 			(at 160.02 53.34 0)
 			(effects
@@
 		)
 	)
+	(embedded_fonts no)
 )
